File: _autosave-power2.kicad_sch (KiCad schematic)
At the start: 26 parts, among them P1 Header 4, P4 Header 4, P5 Header 4, P6 Header 2, U3 TMR 6-2421WIR, U4 LM3940IMP-3.3

Commit message: revised pcb and schematics
Connections:
- net GND: now also C13.2, C20.2, U4.2 (GND), U4.4 (GND)
