File: amplifier.kicad_sch (KiCad schematic)
At the start: 29 parts, among them U7 BUF602xDBV, U8 LT1818CS5-TRMPBF, U9 AD8038AKSZ-REEL7

Commit message: revised pcb and schematics
Parts:
- renumbered RV2 to RV1, U7 to U1, U8 to U2, U9 to U6
Changed lines of the file:
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@@
 (kicad_sch
-	(version 20231120)
+	(version 20250114)
 	(generator "eeschema")
-	(generator_version "8.0")
+	(generator_version "9.0")
 	(paper "A4")
+	(text "make the gain super adjustable over this..  from gain of 1 to 2k because of the bandwidth issues..\n"
+		(exclude_from_sim no)
+		(at 226.568 45.212 0)
+		(effects
+			(font
+				(size 1.27 1.27)
+			)
+		)
+	)
+	(text "The purpose of the first BUF602 is likely to present a\n high-impedance low bias current port to the PMT. It also helps \nwith the impedance matching.\n\n"
+		(exclude_from_sim no)
+		(at 49.022 55.372 0)
+		(effects
+			(font
+				(size 1.27 1.27)
+			)
+		)
+	)
+	(text "When using the LT1818, when using a resistor larger than 500Ohms, a paralel capacitor of value \nCF > RG * Cin/RF should be used to cancel the input pole. Very limited bandwidth at G = -20,\nto increase this switch out the feedback resistor f-3b = 350MHz when G = -1.\n"
+		(exclude_from_sim no)
+		(at 126.238 43.688 0)
+		(effects
+			(font
+				(size 1.27 1.27)
+			)
+		)
+	)
+	(text "Filter is not exactly necessary\n just wanted to have the option\n to configure things. "
+		(exclude_from_sim no)
+		(at 112.522 107.95 0)
+		(effects
+			(font
+				(size 1.27 1.27)
+			)
+		)
+	)
+	(text "This filter is also not necessary\nconsider removing the resistor."
+		(exclude_from_sim no)
+		(at 180.34 109.982 0)
+		(effects
+			(font
+				(size 1.27 1.27)
+			)
+		)
+	)
 	(junction
 		(at 50.8 105.41)
@@
 		)
 	)
-	(text "make the gain super adjustable over this..  from gain of 1 to 2k because of the bandwidth issues..\n"
-		(exclude_from_sim no)
-		(at 226.568 45.212 0)
-		(effects
-			(font
-				(size 1.27 1.27)
-			)
-		)
-	)
-	(text "The purpose of the first BUF602 is likely to present a\n high-impedance low bias current port to the PMT. It also helps \nwith the impedance matching.\n\n"
-		(exclude_from_sim no)
-		(at 49.022 55.372 0)
-		(effects
-			(font
-				(size 1.27 1.27)
-			)
-		)
-	)
-	(text "When using the LT1818, when using a resistor larger than 500Ohms, a paralel capacitor of value \nCF > RG * Cin/RF should be used to cancel the input pole. Very limited bandwidth at G = -20,\nto increase this switch out the feedback resistor f-3b = 350MHz when G = -1.\n"
-		(exclude_from_sim no)
-		(at 126.238 43.688 0)
-		(effects
-			(font
-				(size 1.27 1.27)
-			)
-		)
-	)
-	(text "Filter is not exactly necessary\n just wanted to have the option\n to configure things. "
-		(exclude_from_sim no)
-		(at 112.522 107.95 0)
-		(effects
-			(font
-				(size 1.27 1.27)
-			)
-		)
-	)
-	(text "This filter is also not necessary\nconsider removing the resistor."
-		(exclude_from_sim no)
-		(at 180.34 109.982 0)
-		(effects
-			(font
-				(size 1.27 1.27)
-			)
-		)
-	)
 	(hierarchical_label "VCC_-5V"
 		(shape input)
@@
 		(on_board yes)
 		(dnp no)
-		(property "Reference" "U8"
+		(property "Reference" "U2"
 			(at 125.73 77.47 0)
 			(effects
@@
 		(dnp no)
 		(fields_autoplaced yes)
-		(property "Reference" "U7"
+		(property "Reference" "U1"
 			(at 66.04 83.8514 0)
 			(effects
@@
 		(dnp no)
 		(fields_autoplaced yes)
-		(property "Reference" "RV2"
+		(property "Reference" "RV1"
 			(at 233.68 72.39 90)
 			(effects
@@
 		(on_board yes)
 		(dnp no)
-		(property "Reference" "U9"
+		(property "Reference" "U6"
 			(at 237.49 77.47 0)
 			(effects
