File: discriminator2.kicad_sch (KiCad schematic)
At the start: 6 parts, among them U10 ADCMP601BKSZ-R2

Commit message: revised pcb and schematics
Parts:
- renumbered C19 to C48, C18 to C49, R14 to R30
Changed lines of the file:
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@@
 (kicad_sch
-	(version 20231120)
+	(version 20250114)
 	(generator "eeschema")
-	(generator_version "8.0")
+	(generator_version "9.0")
 	(paper "A4")
+	(text "Minimum pulse width of 4.5ns so in theory could have the bandwidth necessary over the amplifier stage\nif resistors were switched out and be able to reliably trigger. "
+		(exclude_from_sim no)
+		(at 135.128 38.608 0)
+		(effects
+			(font
+				(size 1.27 1.27)
+			)
+		)
+	)
+	(text "does not recommend decoupling caps for this \ngives hysteresis of around 50mV, do we need hysterisis one shot has schmitt trigger inputs"
+		(exclude_from_sim no)
+		(at 256.032 58.42 0)
+		(effects
+			(font
+				(size 1.27 1.27)
+			)
+		)
+	)
+	(text "These resistor values are way too big. Placeholder "
+		(exclude_from_sim no)
+		(at 234.188 84.582 0)
+		(effects
+			(font
+				(size 1.27 1.27)
+			)
+		)
+	)
+	(text "hysteresis\n"
+		(exclude_from_sim no)
+		(at 153.162 48.006 0)
+		(effects
+			(font
+				(size 1.27 1.27)
+			)
+		)
+	)
 	(junction
 		(at 195.58 54.61)
@@
 		)
 	)
-	(text "Minimum pulse width of 4.5ns so in theory could have the bandwidth necessary over the amplifier stage\nif resistors were switched out and be able to reliably trigger. "
-		(exclude_from_sim no)
-		(at 135.128 38.608 0)
-		(effects
-			(font
-				(size 1.27 1.27)
-			)
-		)
-	)
-	(text "does not recommend decoupling caps for this \ngives hysteresis of around 50mV, do we need hysterisis one shot has schmitt trigger inputs"
-		(exclude_from_sim no)
-		(at 256.032 58.42 0)
-		(effects
-			(font
-				(size 1.27 1.27)
-			)
-		)
-	)
-	(text "These resistor values are way too big. Placeholder "
-		(exclude_from_sim no)
-		(at 234.188 84.582 0)
-		(effects
-			(font
-				(size 1.27 1.27)
-			)
-		)
-	)
-	(text "hysteresis\n"
-		(exclude_from_sim no)
-		(at 153.162 48.006 0)
-		(effects
-			(font
-				(size 1.27 1.27)
-			)
-		)
-	)
 	(hierarchical_label "DISC_IN"
 		(shape input)
@@
 		(dnp no)
 		(fields_autoplaced yes)
-		(property "Reference" "R14"
+		(property "Reference" "R30"
 			(at 203.2 59.69 90)
 			(effects
@@
 		(dnp no)
 		(fields_autoplaced yes)
-		(property "Reference" "#PWR052"
+		(property "Reference" "#PWR081"
 			(at 189.23 40.64 0)
 			(effects
@@
 		(dnp no)
 		(fields_autoplaced yes)
-		(property "Reference" "#PWR050"
+		(property "Reference" "#PWR082"
 			(at 201.93 40.64 0)
 			(effects
@@
 		(dnp no)
 		(fields_autoplaced yes)
-		(property "Reference" "C19"
+		(property "Reference" "C48"
 			(at 186.69 52.0638 0)
 			(effects
@@
 		(on_board yes)
 		(dnp no)
-		(property "Reference" "C18"
+		(property "Reference" "C49"
 			(at 199.39 52.0638 0)
 			(effects
@@
 		(dnp no)
 		(fields_autoplaced yes)
-		(property "Reference" "#PWR021"
+		(property "Reference" "#PWR083"
 			(at 204.47 95.25 0)
 			(effects
