File: jumper.kicad_sch (KiCad schematic)
At the start: 3 parts, among them U5 SN74LVC1T45DBV

Commit message: revised pcb and schematics
Parts:
- renumbered C24 to C50, C25 to C51, U5 to U11
Changed lines of the file:
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@@
 (kicad_sch
-	(version 20231120)
+	(version 20250114)
 	(generator "eeschema")
-	(generator_version "8.0")
+	(generator_version "9.0")
 	(paper "A4")
+	(text "Direction from B -> A, input DIR driven L\n"
+		(exclude_from_sim no)
+		(at 165.354 82.804 0)
+		(effects
+			(font
+				(size 1.27 1.27)
+			)
+		)
+	)
 	(junction
 		(at 157.48 119.38)
@@
 			(width 0)
 			(type default)
-		)
-	)
-	(text "Direction from B -> A, input DIR driven L\n"
-		(exclude_from_sim no)
-		(at 165.354 82.804 0)
-		(effects
-			(font
-				(size 1.27 1.27)
-			)
 		)
 	)
@@
 		(on_board yes)
 		(dnp no)
-		(property "Reference" "U5"
+		(property "Reference" "U11"
 			(at 147.32 109.1886 0)
 			(effects
@@
 		(dnp no)
 		(fields_autoplaced yes)
-		(property "Reference" "#PWR027"
+		(property "Reference" "#PWR084"
 			(at 157.48 134.62 0)
 			(effects
@@
 		(dnp no)
 		(fields_autoplaced yes)
-		(property "Reference" "C25"
+		(property "Reference" "C51"
 			(at 175.26 123.1962 0)
 			(effects
@@
 		(dnp no)
 		(fields_autoplaced yes)
-		(property "Reference" "C24"
+		(property "Reference" "C50"
 			(at 160.02 123.1962 0)
 			(effects
@@
 		(dnp no)
 		(fields_autoplaced yes)
-		(property "Reference" "#PWR028"
+		(property "Reference" "#PWR085"
 			(at 172.72 134.62 0)
 			(effects
