File: monostable.kicad_sch (KiCad schematic)
At the start: 4 parts, among them U15 74LVC1G123DCTRE4

Commit message: revised pcb and schematics
Parts:
- renumbered C54 to C52, R33 to R32, U15 to U13
Changed lines of the file:
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@@
 (kicad_sch
-	(version 20231120)
+	(version 20250114)
 	(generator "eeschema")
-	(generator_version "8.0")
+	(generator_version "9.0")
 	(paper "A4")
+	(text "adjust the values of these later for what is coming out of the comparator"
+		(exclude_from_sim no)
+		(at 175.26 39.116 0)
+		(effects
+			(font
+				(size 1.27 1.27)
+			)
+		)
+	)
+	(text "This one-shot is configured to trigger on the rising edge of the input pulse. We want the \noutput pulse to be around 150ns long. As specified by the spec sheet, C = 28pF and R = 2kOhm for a\n Vcc = +5V. If this pulse needs to be longer, the supply voltage needs to be smaller. "
+		(exclude_from_sim no)
+		(at 163.068 112.268 0)
+		(effects
+			(font
+				(size 1.27 1.27)
+			)
+		)
+	)
+	(text "is this wired correctly -- hysteresis?\n"
+		(exclude_from_sim no)
+		(at 156.972 42.672 0)
+		(effects
+			(font
+				(size 1.27 1.27)
+			)
+		)
+	)
+	(text "to lvds"
+		(exclude_from_sim no)
+		(at 226.314 71.12 0)
+		(effects
+			(font
+				(size 1.27 1.27)
+			)
+		)
+	)
 	(junction
 		(at 123.19 86.36)
@@
 		)
 	)
-	(text "adjust the values of these later for what is coming out of the comparator"
-		(exclude_from_sim no)
-		(at 175.26 39.116 0)
-		(effects
-			(font
-				(size 1.27 1.27)
-			)
-		)
-	)
-	(text "This one-shot is configured to trigger on the rising edge of the input pulse. We want the \noutput pulse to be around 150ns long. As specified by the spec sheet, C = 28pF and R = 2kOhm for a\n Vcc = +5V. If this pulse needs to be longer, the supply voltage needs to be smaller. "
-		(exclude_from_sim no)
-		(at 163.068 112.268 0)
-		(effects
-			(font
-				(size 1.27 1.27)
-			)
-		)
-	)
-	(text "is this wired correctly -- hysteresis?\n"
-		(exclude_from_sim no)
-		(at 156.972 42.672 0)
-		(effects
-			(font
-				(size 1.27 1.27)
-			)
-		)
-	)
-	(text "to lvds"
-		(exclude_from_sim no)
-		(at 226.314 71.12 0)
-		(effects
-			(font
-				(size 1.27 1.27)
-			)
-		)
-	)
 	(hierarchical_label "MONO_IN"
 		(shape input)
@@
 		(dnp no)
 		(fields_autoplaced yes)
-		(property "Reference" "C54"
+		(property "Reference" "C52"
 			(at 176.5363 46.99 90)
 			(effects
@@
 		(dnp no)
 		(fields_autoplaced yes)
-		(property "Reference" "U15"
+		(property "Reference" "U13"
 			(at 148.59 60.96 0)
 			(effects
@@
 		(dnp no)
 		(fields_autoplaced yes)
-		(property "Reference" "R33"
+		(property "Reference" "R32"
 			(at 147.32 48.26 90)
 			(effects
