File: output.kicad_sch (KiCad schematic)
At the start: 3 parts, among them U16 SN65LVDS1DBVR

Commit message: revised pcb and schematics
Parts:
- renumbered U16 to U14
Changed lines of the file:
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@@
 (kicad_sch
-	(version 20231120)
+	(version 20250114)
 	(generator "eeschema")
-	(generator_version "8.0")
+	(generator_version "9.0")
 	(paper "A4")
+	(text "These are not the decoupling caps recommmended by the spec sheet -- says it need a 0.1uF and\na 0.001uF polarized capacitor. May need to be AC coupled?"
+		(exclude_from_sim no)
+		(at 170.942 66.548 0)
+		(effects
+			(font
+				(size 1.27 1.27)
+			)
+		)
+	)
+	(text "I'm fairly certain that input signals can be up to 5V."
+		(exclude_from_sim no)
+		(at 147.828 72.39 0)
+		(effects
+			(font
+				(size 1.27 1.27)
+			)
+		)
+	)
 	(junction
 		(at 106.68 81.28)
@@
 			(width 0)
 			(type default)
-		)
-	)
-	(text "These are not the decoupling caps recommmended by the spec sheet -- says it need a 0.1uF and\na 0.001uF polarized capacitor. May need to be AC coupled?"
-		(exclude_from_sim no)
-		(at 170.942 66.548 0)
-		(effects
-			(font
-				(size 1.27 1.27)
-			)
-		)
-	)
-	(text "I'm fairly certain that input signals can be up to 5V."
-		(exclude_from_sim no)
-		(at 147.828 72.39 0)
-		(effects
-			(font
-				(size 1.27 1.27)
-			)
 		)
 	)
@@
 		(dnp no)
 		(fields_autoplaced yes)
-		(property "Reference" "U16"
+		(property "Reference" "U14"
 			(at 133.35 80.01 0)
 			(effects
